Commit message: 修改关节方向

File: src/yj10_description/urdf/yj10.urdf (robot description, URDF)
Before this commit: robot yj10, 7 links, 6 joints
Joints:
- joint joint1: axis 0 0 1 -> 0 0 -1
- joint joint2: axis 0.99995 -0.009646 0 -> -0.99995 0.009646 0
- joint joint3: axis -0.99995 0.009646 0 -> 0.99995 -0.009646 0
- joint joint4: axis 0.99995 -0.009646 0 -> -0.99995 0.009646 0
- joint joint5: axis 0.009646 0.99995 0 -> -0.009646 -0.99995 0

Commit message: 修改 joint axis 误差

File: src/yj10_description/urdf/yj10.urdf (robot description, URDF)
Before this commit: robot yj10, 7 links, 6 joints
Joints:
- joint joint2: axis -0.99995 0.009646 0 -> -1 0 0
- joint joint3: axis 0.99995 -0.009646 0 -> 1 0 0
- joint joint4: axis -0.99995 0.009646 0 -> -1 0 0
- joint joint5: axis -0.009646 -0.99995 0 -> 0 -1 0

Commit message: 键盘控制完成

File: src/yj10_description/urdf/yj10.urdf (robot description, URDF)
Before this commit: robot yj10, 7 links, 6 joints
Joints:
- joint joint1: limit lower=-1.5708 upper=1.5708 effort=10000 velocity=0.2 -> lower=-1.5708 upper=1.5708 effort=10000 velocity=0.4
- joint joint2: limit lower=-1.5708 upper=1.5708 effort=10000 velocity=0.2 -> lower=-1.5708 upper=1.5708 effort=10000 velocity=0.4
- joint joint3: limit lower=-1.5708 upper=1.5708 effort=10000 velocity=0.2 -> lower=-1.5708 upper=1.5708 effort=10000 velocity=0.4
- joint joint4: limit lower=-1.5708 upper=1.5708 effort=10000 velocity=0.2 -> lower=-1.5708 upper=1.5708 effort=10000 velocity=0.4
- joint joint5: limit lower=-1.5708 upper=1.5708 effort=10000 velocity=0.2 -> lower=-1.5708 upper=1.5708 effort=10000 velocity=0.4

Commit message: 实机测试完毕！由于机械臂不能交替读写，所以读取返回假数据

File: src/yj10_description/urdf/yj10.urdf (robot description, URDF)
Before this commit: robot yj10, 7 links, 6 joints
Joints:
- joint joint1: limit lower=-1.5708 upper=1.5708 effort=10000 velocity=0.4 -> lower=-1.5708 upper=1.5708 effort=10000 velocity=0.57
- joint joint2: limit lower=-1.5708 upper=1.5708 effort=10000 velocity=0.4 -> lower=-1.5708 upper=1.5708 effort=10000 velocity=0.57
- joint joint3: limit lower=-1.5708 upper=1.5708 effort=10000 velocity=0.4 -> lower=-1.5708 upper=1.5708 effort=10000 velocity=0.57
- joint joint4: limit lower=-1.5708 upper=1.5708 effort=10000 velocity=0.4 -> lower=-1.5708 upper=1.5708 effort=10000 velocity=0.57
- joint joint5: limit lower=-1.5708 upper=1.5708 effort=10000 velocity=0.4 -> lower=-1.5708 upper=1.5708 effort=10000 velocity=0.57

Commit message: 修改模型和最小容许精度误差，提高控制精度现在大概 5 mm 以内

File: src/yj10_description/urdf/yj10.urdf (robot description, URDF)
Before this commit: robot yj10, 7 links, 6 joints
Joints:
- joint joint2: axis -1 0 0 -> -0.99995 0.009646 0
- joint joint3: axis 1 0 0 -> 0.99995 -0.009646 0
- joint joint4: axis -1 0 0 -> -0.99995 0.009646 0
- joint joint5: axis 0 -1 0 -> -0.009646 -0.99995 0

Commit message: 添加 fake_joint，方便解算

File: src/yj10_description/urdf/yj10.urdf (robot description, URDF)
Before this commit: robot yj10, 7 links, 6 joints
Links:
- added link fake_link6; visual box size=0.01 0.01 0.01
Joints:
- added joint fake_joint6: type continuous, parent link5, child fake_link6, origin xyz=0 0.1 0 rpy=0 0 0, axis 0 0 1

Commit message: 摆正轴的位置；添加joint_group_position_controller

File: src/yj10_description/urdf/yj10.urdf (robot description, URDF)
Before this commit: robot yj10, 8 links, 7 joints
Joints:
- joint fake_joint6: origin xyz=0 0.1 0 rpy=0 0 0 -> xyz=0 0.145 0 rpy=0 0 0
- joint joint2: axis -0.99995 0.009646 0 -> -1 0 0
- joint joint3: axis 0.99995 -0.009646 0 -> 1 0 0
- joint joint4: axis -0.99995 0.009646 0 -> -1 0 0
- joint joint5: axis -0.009646 -0.99995 0 -> 0 -1 0

Commit message: 更新模型

File: src/yj10_description/urdf/yj10.urdf (robot description, URDF)
Before this commit: robot yj10, 8 links, 7 joints
Links:
- link base_link: mass 1.7019 -> 1.70194512971782
Joints:
- joint joint2: origin xyz=0.038998 -0.00037619 0.093 rpy=0 0 0 -> xyz=0.039 0 0.093 rpy=0 0 0
- joint joint3: origin xyz=0.0049998 -4.823E-05 0.6 rpy=0 0 0 -> xyz=0.005 0 0.6 rpy=0 0 0
- joint joint4: origin xyz=0.014287 0.59989 0 rpy=0 0 0 -> xyz=0.0085 0.6 0 rpy=0 0 0
- joint joint5: origin xyz=0.041038 0.055577 0 rpy=0 0 0 -> xyz=0.0405 0.05597 0 rpy=0 0 0

Commit message: 修改 fake_joint6 为 joint6_fake，以解决顺序问题

File: src/yj10_description/urdf/yj10.urdf (robot description, URDF)
Before this commit: robot yj10, 8 links, 7 joints
Joints:
- removed joint fake_joint6
- added joint joint6_fake: type continuous, parent link5, child fake_link6, origin xyz=0 0.145 0 rpy=0 0 0, axis 0 0 1

Commit message: Trying to add yj10_gazebo

File: src/yj10_description/urdf/yj10.urdf (robot description, URDF)
Before this commit: robot yj10, 8 links, 7 joints
Links:
- link fake_link6: mass None -> 0.22539

Commit message: 成功实现 gazebo + ros control + moveit

File: src/yj10_description/urdf/yj10.urdf (robot description, URDF)
Before this commit: robot yj10, 8 links, 7 joints
Links:
- link base_link: mass 1.70194512971782 -> 0.6
- link fake_link6: mass 0.22539 -> 0.01
- link link1: mass 0.87269 -> 0.6
- link link2: mass 3.09 -> 0.6
- link link3: mass 1.8688 -> 0.6
- link link4: mass 0.63938 -> 0.6
- link link5: mass 0.22539 -> 0.6
